File: 1. PCB/3. Stair Light - PSU/stair light psu.brd (EAGLE design)
At the start: 46.5 x 47 mm, 12 parts, among them U1 HILINK HLK-PM01 5V

Commit message: Released v1.0 and sending the boards to manufacture.
Other:
- board text added: "2021/02"
- board text added: "JLCJLCJLCJLC"
- board text added: "STAIR LIGHT PSU"
- board text removed: "2021/01"
- board text removed: "LED STAIRS PSU"
