File: 1. PCB/3. Stair Light - PSU/stair light psu.sch (EAGLE design)
At the start: 12 parts, among them J2 TERMINAL_5MM_4P_90º_20A, J3 1X05, U1 HILINK HLK-PM01 5V

Commit message: Released v1.0 and sending the boards to manufacture.
Other:
- note added: "STAIR LIGHT PSU"
- note removed: "LED STAIRS PSU"
Changed lines of the file:
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@@
 <sheet>
 <plain>
-<text x="163.576" y="24.892" size="5.08" layer="94">LED STAIRS PSU</text>
+<text x="163.576" y="24.892" size="5.08" layer="94">STAIR LIGHT PSU</text>
 <text x="163.576" y="12.192" size="5.08" layer="94">http://giltesa.com</text>
 <text x="243.586" y="6.35" size="2.54" layer="94">V1.0</text>
