File: 1. PCB/1. Stair Light - Controller/stair light controller.brd (EAGLE design)
At the start: 82.9 x 104.1 mm, 60 parts, among them IC2 DS3231/SO, J1 USB-C, Q1 MMBT2222, Q2 MMBT2222, Q3 MMBT2222, U1 ESP32-WROVER-B, U1" ESP32-WROOM, U2 CP2104, U4 HTU21D

Commit message: no message
Parts:
- added 16_RX2, 17_TX2: (no value), SparkFun-Connectors:TP_15TH
- BUZZER: value BUZZER_9MM -> (none)
- IC2: value DS3231/SO -> DS3231
- R3: value 120 -> 120R; device SparkFun:0603 -> ,giltesa:R0603
- SW1: device ,giltesa:JUMPER-SMD-CERRADO_0402 -> ,giltesa:JUMPER-SMD_0402
- moved U$13 104.0 mm to (2.26, 22.7)
- moved U$10 91.2 mm to (87.2, 23.5)
- moved LOGO1 88.5 mm to (7.67, 17.9)
- moved SW2 7.88 mm to (11.0, 33.1), turned to 270 degrees
- moved R11 6.99 mm to (76.5, 36.2), turned to 180 degrees
- moved R3 6.49 mm to (46.6, 28.1)
- moved TP2 5.75 mm to (72.8, 38.1)
- moved TP1 5.75 mm to (62.6, 38.1)
- moved R5 4.83 mm to (76.5, 38.2), turned to 0 degrees
- moved Q1 3.96 mm to (74.5, 42.0)
- moved Q2 3.96 mm to (78.4, 42.0)
- moved SW1 3.77 mm to (62.1, 35.0), turned to 90 degrees
- moved R13 3.30 mm to (3.17, 33.1), turned to 270 degrees
- moved SW3 2.57 mm to (46.6, 26.0)
- moved D1 1.89 mm to (7.11, 32.4), turned to 180 degrees
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- renumbered AMS1117-3.3 to IC3, U$30 to JP2, U$31 to IC1, U4 to U3
Connections:
- net 16_NOT_DEV_PCB_RX2: now also 16_RX2.P$1
- net 17_NOT_DEV_PCB_TX2: now also 17_TX2.P$1
- net 3.3V: now also RN1.1; no longer RN1.2
- net A: now also JP1.3; no longer JP1.4
- net B: now also JP1.4; no longer JP1.3
- net N$1: now also RN1.8; no longer RN1.7
- net N$2: now also RN1.7; no longer RN1.8
- net STAT_LED: now also RN1.2; no longer RN1.1
- net SW_DOWN: now also RN2.2; no longer RN2.3
- net SW_MENU: now also RN2.4; no longer RN2.1
- net SW_OK: now also RN2.1; no longer RN2.4
- net SW_UP: now also RN2.3; no longer RN2.2
Routing:
- net 3.3V: track 7.23 -> 328.3 mm, vias 0 -> 31
- net RX: track 0.00 -> 99.2 mm, vias 0 -> 2
- net RTS: track 0.00 -> 68.2 mm, vias 0 -> 2
- net SDA: track 0.00 -> 53.4 mm, vias 0 -> 2
- net SCL: track 0.00 -> 52.6 mm, vias 0 -> 2
- net N$4: track 0.00 -> 32.0 mm
- net SW_OK: track 0.00 -> 29.9 mm
- net 0: track 0.00 -> 29.4 mm, vias 0 -> 1
- net SW_DOWN: track 0.00 -> 21.6 mm
- net D+: track 0.00 -> 20.5 mm, vias 0 -> 3
- net CHIP_PU: track 0.00 -> 18.3 mm
- net N$6: track 0.00 -> 18.1 mm
- net 5V: track 31.9 -> 49.8 mm
- net TX_LED: track 0.00 -> 15.8 mm
- net RX_LED: track 0.00 -> 14.8 mm, vias 0 -> 2
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- added copper zone on layer 1, net 3.3V
- added copper zone on layer 16, net 3.3V
Other:
- board text added: "2021/01"
- board text added: "STAIR LIGHT CONTROLLER"
- board text added: "V1.0"

Commit message: no message
Parts:
- removed SW1: (no value), ,giltesa:JUMPER-SMD_0402
- removed SW2: (no value), ,giltesa:JUMPER-SMD-CERRADO
- removed SW3: (no value), ,giltesa:JUMPER-SMD
- removed U1: ESP32-WROVER-B, ,giltesa:ESP32-WROVER-B
- removed U2: CP2104, microbuilder:QFN24_4MM_SMSC
- added IC4: MAX3485, SparkFun-DigitalIC:SO08
- added IC5: DS3231, adafruit:SO16W
- added J2: TFT_GC9A01, ,giltesa:LCD_GC9A01
- added JP3: (no value), ,giltesa:JUMPER-SMD_0402
- added X1: USB-C, SparkFun-Connectors:USB-C-16P
- C6, C8: value 22uF -> 10uF; device SparkFun:EIA3528 -> SparkFun:EIA3216
- IC1: value MAX3485 -> ESP32-WROVER-B; device SparkFun-DigitalIC:SO08 -> ,giltesa:ESP32-WROVER-B
- IC2: value DS3231 -> CP2104; device adafruit:SO16W -> microbuilder:QFN24_4MM_SMSC
- IC3: value AMS1117-3.3 -> HT7333; device ,giltesa:SOT223 -> ,giltesa:SOT89_1
- J1: value USB-C -> (none); device SparkFun-Connectors:USB-C-16P -> pinhead:1X05
- JP1: device pinhead:1X05 -> ,giltesa:JUMPER-SMD_0402
- JP2: value TFT_GC9A01 -> (none); device ,giltesa:LCD_GC9A01 -> ,giltesa:JUMPER-SMD
- moved IC2 52.7 mm to (48.3, 10.8)
- moved J1 49.3 mm to (40.3, 16.3)
- moved IC1 45.1 mm to (64.5, 62.1), turned to 0 degrees
- moved U$10 42.1 mm to (54.1, 49.5), flipped to the bottom, turned to 270 degrees
- moved JP2 30.1 mm to (46.6, 27.3)
- moved JP1 28.8 mm to (62.1, 35.0), turned to 90 degrees
- moved R3 3.18 mm to (46.6, 24.9)
- moved IC3 1.40 mm to (27.2, 24.3)
- moved BAT 0.76 mm to (33.8, 42.0)
- moved U$5 0.76 mm to (33.8, 42.0)
- renumbered U$2 to X2, U3 to IC6
Connections:
- new net N$3: IC3.4
- net 0: now also IC1.25; no longer U1.25
- net 12: now also IC1.14; no longer U1.14
- net 16_NOT_DEV_PCB_RX2: now also IC1.27; no longer U1.27
- net 17_NOT_DEV_PCB_TX2: now also IC1.28; no longer U1.28
- net 3.3V: now also IC1.2, IC2.5, IC2.6, IC2.7, IC3.3, IC4.8, IC5.2, J2.3V3, J2.3V3"; no longer IC1.8, IC2.2, IC3.2, IC3.4, JP2.3V3, JP2.3V3", U1.2, U2.5, U2.6, U2.7
- net 5V: now also IC2.8, IC3.2, J1.1; no longer IC3.3, JP1.1, U2.8
- net A: now also IC4.6, J1.3, JP2.1; no longer IC1.6, JP1.3, SW3.1
- net B: now also IC4.7, J1.4; no longer IC1.7, JP1.4
- net BUZZER: now also IC1.30; no longer U1.30
- net CHIP_PU: now also IC1.3; no longer U1.3
- net D+: now also IC2.3; no longer U2.3
- net D-: now also IC2.4; no longer U2.4
- net DTR: now also IC2.23; no longer U2.23
- net EXT_PCB_5V: now also X1.VBUS1, X1.VBUS2; no longer J1.VBUS1, J1.VBUS2
- net EXT_PCB_CC1: now also X1.A5; no longer J1.A5
- net EXT_PCB_CC2: now also X1.B5; no longer J1.B5
- net EXT_PCB_D+: now also X1.A6, X1.B6; no longer J1.A6, J1.B6
- net EXT_PCB_D-: now also X1.A7, X1.B7; no longer J1.A7, J1.B7
- net EXT_PCB_GND: now also X1.GND, X1.GND2; no longer J1.GND, J1.GND2
- net GND: now also IC1.1, IC1.15, IC1.38, IC1.GND, IC2.2, IC2.THERM, IC4.5, IC5.10, IC5.11, IC5.12, IC5.13, IC5.5, IC5.6, IC5.7, IC5.8, IC5.9, J1.5, J2.GND, J2.GND", JP1.2; no longer IC1.5, IC2.10, IC2.11, IC2.12, IC2.13, IC2.5, IC2.6, IC2.7, IC2.8, IC2.9, JP1.5, JP2.GND, JP2.GND", SW1.2, U1.1, U1.15, U1.38, U1.GND, U2.2, U2.THERM
- net MISO: now also IC1.24; no longer U1.24
- net MOSI: now also IC1.23, J2.SDA, J2.SDA"; no longer JP2.SDA, JP2.SDA", U1.23
- net N$13: now also JP1.1; no longer SW1.1
- net N$14: now also JP2.2; no longer SW3.2
- net N$18: now also IC1.32; no longer U1.32
- net N$27: now also IC1.20; no longer U1.20
- net N$28: now also IC1.19; no longer U1.19
- net N$29: now also IC1.22; no longer U1.22
- net N$30: now also IC1.21; no longer U1.21
- net N$33: now also IC1.17; no longer U1.17
- net N$34: now also IC1.18; no longer U1.18
- net N$35: now also JP3.2; no longer SW2.2
- net N$4: now also IC5.14, JP3.1; no longer IC2.14, SW2.1
- net NEOPIXEL: now also IC1.31, J1.2; no longer JP1.2, U1.31
- net RS485_CS: now also IC1.8, IC4.2, IC4.3; no longer IC1.2, IC1.3, U1.8
- net RS485_RX: now also IC1.11, IC4.1; no longer IC1.1, U1.11
- net RS485_TX: now also IC1.10, IC4.4; no longer IC1.4, U1.10
- net RTS: now also IC2.19; no longer U2.19
- net RX: now also IC1.35, IC2.20; no longer U1.35, U2.20
- net RX_LED: now also IC2.13; no longer U2.13
- net SCK: now also IC1.13, J2.SCL, J2.SCL"; no longer JP2.SCL, JP2.SCL", U1.13
- net SCL: now also IC1.36, IC5.16; no longer IC2.16, U1.36
- net SDA: now also IC1.33, IC5.15; no longer IC2.15, U1.33
- net SD_CS: now also IC1.16; no longer U1.16
- net STAT_LED: now also IC1.29; no longer U1.29
- net SW_DOWN: now also IC1.4; no longer U1.4
- net SW_MENU: now also IC1.6; no longer U1.6
- net SW_OK: now also IC1.5; no longer U1.5
- net SW_UP: now also IC1.7; no longer U1.7
- net TFT_BLK: now also IC1.37, J2.BLK, J2.BLK"; no longer JP2.BLK, JP2.BLK", U1.37
- net TFT_CS: now also IC1.26, J2.CS, J2.CS"; no longer JP2.CS, JP2.CS", U1.26
- net TFT_DC: now also IC1.12, J2.DC, J2.DC"; no longer JP2.DC, JP2.DC", U1.12
- net TFT_RST: now also IC1.9, J2.RST, J2.RST"; no longer JP2.RST, JP2.RST", U1.9
- net TX: now also IC1.34, IC2.21; no longer U1.34, U2.21
- net TX_LED: now also IC2.14; no longer U2.14
Routing:
- net SCL: track 52.6 -> 168.0 mm, vias 2 -> 5
- net MOSI: track 5.68 -> 116.9 mm, vias 0 -> 4
- net SDA: track 53.4 -> 162.8 mm, vias 2 -> 5
- net SCK: track 0.77 -> 100.4 mm, vias 0 -> 4
- net TX: track 0.26 -> 97.2 mm, vias 0 -> 2
- net BUZZER: track 0.26 -> 94.5 mm, vias 0 -> 4
- net MISO: track 2.88 -> 89.9 mm, vias 0 -> 3
- net NEOPIXEL: track 0.26 -> 81.9 mm, vias 0 -> 3
- net SD_CS: track 5.17 -> 76.5 mm, vias 0 -> 3
- net DTR: track 5.79 -> 67.5 mm, vias 0 -> 2
- net STAT_LED: track 0.26 -> 61.9 mm, vias 0 -> 4
- net TFT_CS: track 0.77 -> 59.9 mm, vias 0 -> 2
- net RS485_CS: track 0.26 -> 54.1 mm, vias 0 -> 2
- net CHIP_PU: track 18.3 -> 70.9 mm, vias 0 -> 3
- net RS485_TX: track 0.26 -> 50.3 mm, vias 0 -> 2
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- added copper zone on layer 1, net N$3
- added copper zone on layer 16, net N$3
- removed copper zone on layer 1, net 3.3V
- removed copper zone on layer 16, net 3.3V
Other:
- board text added: "2021/02"
- board text removed: "2021/01"

Commit message: Released v1.0 and sending the boards to manufacture.
Parts:
- D1: value 1N4148 -> 1N4148
- moved RN3 0.13 mm to (47.0, -15.7)
Other:
- board size 82.9 x 104.1 mm -> 82.9 x 104.3 mm
- board text added: "JLCJLCJLCJLC"

Commit message: no message
Parts:
- removed RN3: 10k, resistor-dil:0603-ARV
Connections:
- net EXT_PCB_3.3V: no longer RN3.1, RN3.2, RN3.3, RN3.4
- net EXT_PCB_MISO: no longer RN3.8
- net EXT_PCB_MOSI: no longer RN3.6
- net EXT_PCB_SCK: no longer RN3.7
- net EXT_PCB_SD_CS: no longer RN3.5
Routing:
- net EXT_PCB_3.3V: track 32.7 -> 19.9 mm
- net EXT_PCB_SCK: track 15.9 -> 10.2 mm
- net EXT_PCB_MOSI: track 16.2 -> 11.5 mm
- net EXT_PCB_SD_CS: track 17.9 -> 13.3 mm
- net EXT_PCB_MISO: track 18.1 -> 13.9 mm
Changed lines of the file:
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@@
 <layer number="20" name="Dimension" color="15" fill="1" visible="yes" active="yes"/>
 <layer number="21" name="tPlace" color="7" fill="1" visible="yes" active="yes"/>
-<layer number="22" name="bPlace" color="7" fill="1" visible="yes" active="yes"/>
-<layer number="23" name="tOrigins" color="15" fill="1" visible="no" active="yes"/>
+<layer number="22" name="bPlace" color="7" fill="1" visible="no" active="yes"/>
+<layer number="23" name="tOrigins" color="15" fill="1" visible="yes" active="yes"/>
 <layer number="24" name="bOrigins" color="15" fill="1" visible="no" active="yes"/>
 <layer number="25" name="tNames" color="7" fill="1" visible="no" active="yes"/>
@@
 <attribute name="VALUE" x="24.676" y="76.708" size="1.016" layer="21" font="vector" ratio="16" align="center-left"/>
 </element>
-<element name="RN3" library="resistor-dil" package="0603-ARV" value="10k" x="46.99" y="-15.748" smashed="yes" rot="R270">
-<attribute name="OC_NEWARK" value="unknown" x="46.99" y="-15.748" size="1.778" layer="27" rot="R270" display="off"/>
-<attribute name="MPN" value="" x="46.99" y="-15.748" size="1.778" layer="27" rot="R270" display="off"/>
-<attribute name="MF" value="" x="46.99" y="-15.748" size="1.778" layer="27" rot="R270" display="off"/>
-<attribute name="OC_FARNELL" value="unknown" x="46.99" y="-15.748" size="1.778" layer="27" rot="R270" display="off"/>
-<attribute name="NAME" x="47.244" y="-13.335" size="0.9144" layer="21" font="vector" ratio="16" align="center"/>
-<attribute name="VALUE" x="45.974" y="-18.161" size="1.016" layer="27" font="vector" ratio="16" align="center-left"/>
-</element>
 <element name="R3" library=",giltesa" package="R0603" value="120R" x="46.609" y="24.892" smashed="yes">
 <attribute name="NAME" x="46.609" y="23.622" size="1.016" layer="21" font="vector" ratio="16" align="center"/>
@@
 <signal name="EXT_PCB_SD_CS">
 <contactref element="X2" pad="2-CS"/>
-<contactref element="RN3" pad="5"/>
 <contactref element="J-SD-E" pad="1"/>
 <wire x1="53.086" y1="-12.446" x2="55.372" y2="-12.446" width="0.3048" layer="1"/>
 <wire x1="55.372" y1="-12.446" x2="57.2036" y2="-10.6144" width="0.3048" layer="1"/>
 <wire x1="57.2036" y1="-9.3709" x2="57.2036" y2="-10.6144" width="0.3048" layer="1"/>
-<wire x1="50.349" y1="-16.948" x2="51.181" y2="-17.78" width="0.3048" layer="1"/>
-<wire x1="51.181" y1="-17.78" x2="52.705" y2="-17.78" width="0.3048" layer="1"/>
-<wire x1="47.615" y1="-16.948" x2="48.584" y2="-16.948" width="0.3048" layer="1"/>
-<wire x1="48.584" y1="-16.948" x2="53.086" y2="-12.446" width="0.3048" layer="1"/>
-<wire x1="50.349" y1="-16.948" x2="48.584" y2="-16.948" width="0.3048" layer="1"/>
+<wire x1="51.251" y1="-14.281" x2="53.086" y2="-12.446" width="0.3048" layer="1"/>
+<wire x1="51.251" y1="-14.281" x2="51.251" y2="-17.215" width="0.3048" layer="1"/>
+<wire x1="51.251" y1="-17.215" x2="51.816" y2="-17.78" width="0.3048" layer="1"/>
+<wire x1="51.816" y1="-17.78" x2="52.705" y2="-17.78" width="0.3048" layer="1"/>
 </signal>
 <signal name="EXT_PCB_MOSI">
 <contactref element="X2" pad="3-DI"/>
-<contactref element="RN3" pad="6"/>
 <contactref element="J-SD-E" pad="2"/>
 <wire x1="52.832" y1="-11.811" x2="54.991" y2="-11.811" width="0.3048" layer="1"/>
 <wire x1="54.991" y1="-11.811" x2="56.1036" y2="-10.6984" width="0.3048" layer="1"/>
 <wire x1="56.1036" y1="-9.3709" x2="56.1036" y2="-10.6984" width="0.3048" layer="1"/>
-<wire x1="47.615" y1="-16.148" x2="48.495" y2="-16.148" width="0.3048" layer="1"/>
-<wire x1="48.495" y1="-16.148" x2="51.1175" y2="-13.5255" width="0.3048" layer="1"/>
-<wire x1="51.1175" y1="-13.5255" x2="52.832" y2="-11.811" width="0.3048" layer="1"/>
 <via x="50.673" y="-13.208" extent="1-16" drill="0.3556"/>
 <wire x1="50.673" y1="-13.208" x2="51.816" y2="-13.208" width="0.3048" layer="16"/>
@@
 <wire x1="52.705" y1="-14.097" x2="52.705" y2="-15.24" width="0.3048" layer="16"/>
 <wire x1="50.673" y1="-13.208" x2="50.8" y2="-13.208" width="0.3048" layer="1"/>
-<wire x1="50.8" y1="-13.208" x2="51.1175" y2="-13.5255" width="0.3048" layer="1"/>
+<wire x1="52.832" y1="-11.811" x2="51.435" y2="-13.208" width="0.3048" layer="1"/>
+<wire x1="51.435" y1="-13.208" x2="50.673" y2="-13.208" width="0.3048" layer="1"/>
 </signal>
 <signal name="EXT_PCB_SCK">
 <contactref element="X2" pad="5-SCK"/>
-<contactref element="RN3" pad="7"/>
 <contactref element="J-SD-E" pad="4"/>
 <wire x1="52.07" y1="-11.176" x2="53.594" y2="-11.176" width="0.3048" layer="1"/>
 <wire x1="53.594" y1="-11.176" x2="53.9036" y2="-10.8664" width="0.3048" layer="1"/>
 <wire x1="53.9036" y1="-9.3709" x2="53.9036" y2="-10.8664" width="0.3048" layer="1"/>
-<wire x1="47.615" y1="-15.348" x2="48.406" y2="-15.348" width="0.3048" layer="1"/>
-<wire x1="48.406" y1="-15.348" x2="49.784" y2="-13.97" width="0.3048" layer="1"/>
-<wire x1="49.784" y1="-13.97" x2="49.784" y2="-12.827" width="0.3048" layer="1"/>
-<wire x1="49.784" y1="-12.827" x2="50.673" y2="-11.938" width="0.3048" layer="1"/>
-<wire x1="52.07" y1="-11.176" x2="51.308" y2="-11.938" width="0.3048" layer="1"/>
-<wire x1="51.308" y1="-11.938" x2="51.181" y2="-11.938" width="0.3048" layer="1"/>
-<wire x1="51.181" y1="-11.938" x2="50.673" y2="-11.938" width="0.3048" layer="1"/>
+<wire x1="52.07" y1="-11.176" x2="51.181" y2="-12.065" width="0.3048" layer="1"/>
 <via x="51.181" y="-12.192" extent="1-16" drill="0.3556"/>
-<wire x1="51.181" y1="-12.192" x2="51.181" y2="-11.938" width="0.3048" layer="1"/>
 <wire x1="55.245" y1="-15.24" x2="54.864" y2="-15.24" width="0.3048" layer="16"/>
 <wire x1="54.864" y1="-15.24" x2="51.816" y2="-12.192" width="0.3048" layer="16"/>
 <wire x1="51.816" y1="-12.192" x2="51.181" y2="-12.192" width="0.3048" layer="16"/>
+<wire x1="51.181" y1="-12.192" x2="51.181" y2="-12.065" width="0.3048" layer="1"/>
 </signal>
 <signal name="EXT_PCB_MISO">
 <contactref element="X2" pad="7-DO"/>
-<contactref element="RN3" pad="8"/>
 <contactref element="J-SD-E" pad="6"/>
-<wire x1="47.615" y1="-14.548" x2="48.317" y2="-14.548" width="0.3048" layer="1"/>
-<wire x1="48.317" y1="-14.548" x2="49.022" y2="-13.843" width="0.3048" layer="1"/>
-<wire x1="49.022" y1="-13.843" x2="49.022" y2="-12.7" width="0.3048" layer="1"/>
 <wire x1="50.419" y1="-11.303" x2="51.054" y2="-11.303" width="0.3048" layer="1"/>
 <wire x1="51.054" y1="-11.303" x2="51.7036" y2="-10.6534" width="0.3048" layer="1"/>
@@
 <wire x1="53.975" y1="-13.335" x2="51.943" y2="-11.303" width="0.3048" layer="16"/>
 <via x="49.53" y="-11.684" extent="1-16" drill="0.3556"/>
-<wire x1="49.022" y1="-12.7" x2="49.784" y2="-11.938" width="0.3048" layer="1"/>
-<wire x1="49.784" y1="-11.938" x2="50.419" y2="-11.303" width="0.3048" layer="1"/>
-<wire x1="49.53" y1="-11.684" x2="49.784" y2="-11.938" width="0.3048" layer="1"/>
+<wire x1="50.038" y1="-11.684" x2="50.419" y2="-11.303" width="0.3048" layer="1"/>
 <wire x1="51.943" y1="-11.303" x2="50.419" y2="-11.303" width="0.3048" layer="16"/>
 <wire x1="50.419" y1="-11.303" x2="50.038" y2="-11.684" width="0.3048" layer="16"/>
 <wire x1="50.038" y1="-11.684" x2="49.53" y2="-11.684" width="0.3048" layer="16"/>
+<wire x1="49.53" y1="-11.684" x2="50.038" y2="-11.684" width="0.3048" layer="1"/>
 </signal>
 <signal name="EXT_PCB_3.3V">
-<contactref element="RN3" pad="1"/>
-<contactref element="RN3" pad="4"/>
-<contactref element="RN3" pad="3"/>
-<contactref element="RN3" pad="2"/>
 <contactref element="X2" pad="4-VCC"/>
 <contactref element="J-SD-E" pad="3"/>
-<wire x1="46.365" y1="-14.548" x2="46.365" y2="-15.348" width="0.4064" layer="1"/>
-<wire x1="46.365" y1="-15.348" x2="46.365" y2="-16.148" width="0.4064" layer="1"/>
-<wire x1="46.365" y1="-16.148" x2="46.365" y2="-16.948" width="0.4064" layer="1"/>
-<wire x1="46.365" y1="-16.948" x2="46.365" y2="-17.409" width="0.4064" layer="1"/>
-<wire x1="46.365" y1="-17.409" x2="46.736" y2="-17.78" width="0.4064" layer="1"/>
-<wire x1="46.736" y1="-17.78" x2="49.784" y2="-17.78" width="0.4064" layer="1"/>
-<wire x1="49.784" y1="-17.78" x2="51.308" y2="-19.304" width="0.4064" layer="1"/>
 <wire x1="58.801" y1="-19.304" x2="59.563" y2="-18.542" width="0.4064" layer="1"/>
 <via x="59.563" y="-12.319" extent="1-16" drill="0.4572"/>
@@
 <wire x1="54.991" y1="-8.636" x2="54.991" y2="-9.3583" width="0.4064" layer="1"/>
 <wire x1="54.991" y1="-9.3583" x2="55.0036" y2="-9.3709" width="0.4064" layer="1"/>
-<wire x1="58.801" y1="-19.304" x2="55.372" y2="-19.304" width="0.4064" layer="1"/>
-<wire x1="55.372" y1="-19.304" x2="51.308" y2="-19.304" width="0.4064" layer="1"/>
-<wire x1="55.245" y1="-17.78" x2="55.245" y2="-19.177" width="0.4064" layer="1"/>
-<wire x1="55.245" y1="-19.177" x2="55.372" y2="-19.304" width="0.4064" layer="1"/>
+<wire x1="58.801" y1="-19.304" x2="55.626" y2="-19.304" width="0.4064" layer="1"/>
+<wire x1="55.245" y1="-17.78" x2="55.245" y2="-18.923" width="0.4064" layer="1"/>
+<wire x1="55.245" y1="-18.923" x2="55.626" y2="-19.304" width="0.4064" layer="1"/>
 <wire x1="57.023" y1="-8.509" x2="55.118" y2="-8.509" width="0.4064" layer="16"/>
 <wire x1="55.118" y1="-8.509" x2="54.991" y2="-8.636" width="0.4064" layer="16"/>
