File: 1. PCB/1. Stair Light - Controller/stair light controller.sch (EAGLE design)
At the start: 60 parts, among them IC2 DS3231/SO, J1 USB-C, Q1 MMBT2222, Q2 MMBT2222, Q3 MMBT2222, SW1 JUMPER-SMD-CERRADO0402, SW2 JUMPER-SMD-CERRADO0805, SW3 JUMPER-SMD0805, U1 ESP32-WROVER-B, U1" ESP32-WROOM, U2 CP2104, U4 HTU21D

Commit message: no message
Parts:
- added 16_RX2, 17_TX2: TEST-POINTTP_15TH_THRU, SparkFun-Connectors:TEST-POINTTP_15TH_THRU
- IC2: value DS3231/SO -> DS3231
- R3: value 120 -> 120R; device SparkFun:RESISTOR0603 -> ,giltesa:R0603
- SW1: value JUMPER-SMD-CERRADO0402 -> JUMPER-SMD0402; device ,giltesa:JUMPER-SMD-CERRADO0402 -> ,giltesa:JUMPER-SMD0402
- renumbered AMS1117-3.3 to IC3, U$30 to JP2, U$31 to IC1, U4 to U3
Connections:
- net 16_NOT_DEV_PCB_RX2: now also 16_RX2.1
- net 17_NOT_DEV_PCB_TX2: now also 17_TX2.1
- net 3.3V: now also RN1A.1; no longer RN1B.1
- net A: now also JP1.3; no longer JP1.4
- net B: now also JP1.4; no longer JP1.3
- net N$1: now also RN1A.2; no longer RN1B.2
- net N$2: now also RN1B.2; no longer RN1A.2
- net STAT_LED: now also RN1B.1; no longer RN1A.1
- net SW_DOWN: now also RN2B.1; no longer RN2C.1
- net SW_MENU: now also RN2D.1; no longer RN2A.1
- net SW_OK: now also RN2A.1; no longer RN2D.1
- net SW_UP: now also RN2C.1; no longer RN2B.1
Other:
- moved on the sheet: RN1A, RN1B, RN2A, RN2B, RN2C, RN2D

Commit message: no message
Parts:
- removed SW1: JUMPER-SMD0402, ,giltesa:JUMPER-SMD0402
- removed SW2: JUMPER-SMD-CERRADO0805, ,giltesa:JUMPER-SMD-CERRADO0805
- removed SW3: JUMPER-SMD0805, ,giltesa:JUMPER-SMD0805
- removed U1: ESP32-WROVER-B, ,giltesa:ESP32-WROVER-B
- removed U2: CP2104, microbuilder:CP2104
- added IC4: MAX3485, SparkFun-DigitalIC:RS485SOIC
- added IC5: DS3231, adafruit:DS3231/SO
- added J2: TFT_GC9A01, ,giltesa:LCD_GC9A01
- added JP3: JUMPER-SMD0402, ,giltesa:JUMPER-SMD0402
- added X1: USB-C, SparkFun-Connectors:USB_C16PIN
- C6, C8: value 22uF -> 10uF; device SparkFun:CAP_POL3528 -> SparkFun:CAP_POL1206
- IC1: value MAX3485 -> ESP32-WROVER-B; device SparkFun-DigitalIC:RS485SOIC -> ,giltesa:ESP32-WROVER-B
- IC2: value DS3231 -> CP2104; device adafruit:DS3231/SO -> microbuilder:CP2104
- IC3: value AMS1117-3.3 -> HT7333; device ,giltesa:AMS1117SOT223 -> ,giltesa:HT7333
- J1: value USB-C -> (none); device SparkFun-Connectors:USB_C16PIN -> pinhead:PINHD-1X5
- JP1: value (none) -> JUMPER-SMD0402; device pinhead:PINHD-1X5 -> ,giltesa:JUMPER-SMD0402
- JP2: value TFT_GC9A01 -> JUMPER-SMD0805; device ,giltesa:LCD_GC9A01 -> ,giltesa:JUMPER-SMD0805
- renumbered U$2 to X2, U3 to IC6
Connections:
- new net N$3: IC3.NC
- net 0: now also IC1.IO0; no longer U1.IO0
- net 12: now also IC1.IO12; no longer U1.IO12
- net 16_NOT_DEV_PCB_RX2: now also IC1.IO16; no longer U1.IO16
- net 17_NOT_DEV_PCB_TX2: now also IC1.IO17; no longer U1.IO17
- net 3.3V: now also IC1.3V3, IC2G$1.REGIN, IC2G$1.VDD, IC2G$1.VIO, IC4.VCC, IC5.VCC, J2.3V3; no longer IC1.VCC, IC2.VCC, IC3.NC, JP2.3V3, U1.3V3, U2G$1.REGIN, U2G$1.VDD, U2G$1.VIO
- net 5V: now also IC2G$1.VBUS, J1.1; no longer JP1.1, U2G$1.VBUS
- net A: now also IC4.A, J1.3, JP2.1; no longer IC1.A, JP1.3, SW3.1
- net B: now also IC4.B, J1.4; no longer IC1.B, JP1.4
- net BUZZER: now also IC1.IO18; no longer U1.IO18
- net CHIP_PU: now also IC1.EN; no longer U1.EN
- net D+: now also IC2G$1.D+; no longer U2G$1.D+
- net D-: now also IC2G$1.D-; no longer U2G$1.D-
- net DTR: now also IC2G$1.DTR; no longer U2G$1.DTR
- net EXT_PCB_5V: now also X1.VBUS; no longer J1.VBUS
- net EXT_PCB_CC1: now also X1.CC1; no longer J1.CC1
- net EXT_PCB_CC2: now also X1.CC2; no longer J1.CC2
- net EXT_PCB_D+: now also X1.D+; no longer J1.D+
- net EXT_PCB_D-: now also X1.D-; no longer J1.D-
- net EXT_PCB_GND: now also X1.GND; no longer J1.GND
- net GND: now also IC1.GND@1, IC1.GND@15, IC1.GND@38, IC2G$1.GND, IC2G$2.TP, IC4.GND, IC5.GND, IC5.NC, IC5.NC1, IC5.NC2, IC5.NC3, IC5.NC4, IC5.NC5, IC5.NC6, IC5.NC7, J1.5, J2.GND, JP1.2; no longer IC2.GND, IC2.NC, IC2.NC1, IC2.NC2, IC2.NC3, IC2.NC4, IC2.NC5, IC2.NC6, IC2.NC7, JP1.5, JP2.GND, SW1.2, U1.GND, U1.GND@1, U1.GND@15, U1.GND@38, U2G$1.GND, U2G$2.TP
- net MISO: now also IC1.IO2; no longer U1.IO2
- net MOSI: now also IC1.IO15, J2.SDA; no longer JP2.SDA, U1.IO15
- net N$13: now also JP1.1; no longer SW1.1
- net N$14: now also JP2.2; no longer SW3.2
- net N$18: now also IC1.IO20; no longer U1.IO20
- net N$27: now also IC1.SCK; no longer U1.SCK
- net N$28: now also IC1.SCS; no longer U1.SCS
- net N$29: now also IC1.SDI; no longer U1.SDI
- net N$30: now also IC1.SDO; no longer U1.SDO
- net N$33: now also IC1.SHD; no longer U1.SHD
- net N$34: now also IC1.SWP; no longer U1.SWP
- net N$35: now also JP3.2; no longer SW2.2
- net N$4: now also IC5.VBAT, JP3.1; no longer IC2.VBAT, SW2.1
- net NEOPIXEL: now also IC1.IO19, J1.2; no longer JP1.2, U1.IO19
- net RS485_CS: now also IC1.IO32, IC4./RE, IC4.DE; no longer IC1./RE, IC1.DE, U1.IO32
- net RS485_RX: now also IC1.IO26, IC4.RO; no longer IC1.RO, U1.IO26
- net RS485_TX: now also IC1.IO25, IC4.DI; no longer IC1.DI, U1.IO25
- net RTS: now also IC2G$1.RTS; no longer U2G$1.RTS
- net RX: now also IC1.TXD, IC2G$1.RXD; no longer U1.TXD, U2G$1.RXD
- net RX_LED: now also IC2G$1.GPIO1/RXLED; no longer U2G$1.GPIO1/RXLED
- net SCK: now also IC1.IO14, J2.SCL; no longer JP2.SCL, U1.IO14
- net SCL: now also IC1.IO22, IC5.SCL; no longer IC2.SCL, U1.IO22
- net SDA: now also IC1.IO21, IC5.SDA; no longer IC2.SDA, U1.IO21
- net SD_CS: now also IC1.IO13; no longer U1.IO13
- net STAT_LED: now also IC1.IO5; no longer U1.IO5
- net SW_DOWN: now also IC1.SENSOR_VP; no longer U1.SENSOR_VP
- net SW_MENU: now also IC1.IO34; no longer U1.IO34
- net SW_OK: now also IC1.SENSOR_VN; no longer U1.SENSOR_VN
- net SW_UP: now also IC1.IO35; no longer U1.IO35
- net TFT_BLK: now also IC1.IO23, J2.BLK; no longer JP2.BLK, U1.IO23
- net TFT_CS: now also IC1.IO4, J2.CS; no longer JP2.CS, U1.IO4
- net TFT_DC: now also IC1.IO27, J2.DC; no longer JP2.DC, U1.IO27
- net TFT_RST: now also IC1.IO33, J2.RST; no longer JP2.RST, U1.IO33
- net TX: now also IC1.RXD, IC2G$1.TXD; no longer U1.RXD, U2G$1.TXD
- net TX_LED: now also IC2G$1.GPIO0/TXLED; no longer U2G$1.GPIO0/TXLED

Commit message: Released v1.0 and sending the boards to manufacture.
Parts:
- D1: value 1N4148 -> 1N4148
Changed lines of the file:
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@@
 <setting verticaltext="up"/>
 </settings>
-<grid distance="100" unitdist="mil" unit="mil" style="lines" multiple="1" display="no" altdistance="0.01" altunitdist="inch" altunit="inch"/>
+<grid distance="0.1" unitdist="inch" unit="inch" style="lines" multiple="1" display="no" altdistance="0.01" altunitdist="inch" altunit="inch"/>
 <layers>
 <layer number="1" name="Top" color="4" fill="1" visible="no" active="no"/>
@@
 <part name="GND8" library="SparkFun" deviceset="GND" device=""/>
 <part name="BAT" library=",giltesa" deviceset="LIR2032_SMD" device="" value="LIR2032"/>
-<part name="D1" library="adafruit" deviceset="DIODE" device="SOD-123" value="1N4148 "/>
+<part name="D1" library="adafruit" deviceset="DIODE" device="SOD-123" value="1N4148"/>
 <part name="R13" library=",giltesa" deviceset="R0603" device="" value="200R"/>
 <part name="JP3" library=",giltesa" deviceset="JUMPER-SMD" device="0402" value=""/>
@@
 <wire x1="292.1" y1="22.86" x2="289.56" y2="22.86" width="0.1524" layer="91"/>
 <junction x="289.56" y="22.86"/>
-<pinref part="S4" gate="G$1" pin="1"/>
-<wire x1="292.1" y1="30.48" x2="289.56" y2="30.48" width="0.1524" layer="91"/>
 <pinref part="S3" gate="G$1" pin="1"/>
 <wire x1="292.1" y1="38.1" x2="289.56" y2="38.1" width="0.1524" layer="91"/>
 <junction x="289.56" y="38.1"/>
 <pinref part="SUPPLY6" gate="G$1" pin="3.3V"/>
+<pinref part="S4" gate="G$1" pin="1"/>
+<wire x1="292.1" y1="30.48" x2="289.56" y2="30.48" width="0.1524" layer="91"/>
+<junction x="289.56" y="30.48"/>
 </segment>
 <segment>
@@
 <pinref part="U1&quot;" gate="G$1" pin="IO2"/>
 <pinref part="IC1" gate="G$1" pin="IO2"/>
+<label x="66.04" y="71.12" size="1.27" layer="95" xref="yes"/>
 <wire x1="60.96" y1="71.12" x2="66.04" y2="71.12" width="0.1524" layer="91"/>
-<label x="66.04" y="71.12" size="1.27" layer="95" xref="yes"/>
+<junction x="60.96" y="71.12"/>
 </segment>
 <segment>
@@
 </sheet>
 </sheets>
+<errors>
+</errors>
 </schematic>
 </drawing>

Commit message: no message
Parts:
- removed RN3: 10k, resistor-dil:4R-N0603-ARV
Connections:
- net EXT_PCB_3.3V: no longer RN3A.1, RN3B.1, RN3C.1, RN3D.1
- net EXT_PCB_MISO: no longer RN3A.2
- net EXT_PCB_MOSI: no longer RN3C.2
- net EXT_PCB_SCK: no longer RN3B.2
- net EXT_PCB_SD_CS: no longer RN3D.2
Other:
- note added: "V1.1"
- note removed: "V1.0"
- moved on the sheet: J-SD, J-SD-E, X2
